Commit message: Hook in AX12 code to use real joint angles in rviz Fix up urdf to have correct axes for all the joints, link sizes and angle precision are still wrong though

File: trunk/utilities/ROS/awesomeo_controller/TypeA.xacro (robot description, xacro)
@@ -1,5 +1,5 @@
 <?xml version="1.0"?>
 <robot name="awesome-o" xmlns:xacro="http://www.ros.org/wiki/xacro">
-<xacro:macro name="arm" params="prefix reflect">
+<xacro:macro name="arm" params="prefix reflect base">
 <link name="${prefix}_shoulder">
 <visual>
@@ -13,9 +13,9 @@
 </visual>
 </link>
-<joint name="base_to_${prefix}_shoulder" type="revolute">
+<joint name="${base+1}:base_to_${prefix}_shoulder" type="revolute">
 <parent link="base_link"/>
 <child link="${prefix}_shoulder"/>
-<origin rpy="0 0 0" xyz="${reflect*0.070} 0 0.03"/>
-<axis xyz="1 0 0"/>
+<origin rpy="1.5 0 0" xyz="${reflect*0.070} 0 0.03"/>
+<axis xyz="${reflect} 0 0"/>
 <limit effort="1000.0" lower="-3.14" upper="3.14" velocity="0.5"/>
 </joint>
@@ -32,9 +32,9 @@
     </visual>
 </link>
-  <joint name="${prefix}_shoulder_to_upper" type="revolute">
+  <joint name="${base+3}:${prefix}_shoulder_to_upper" type="revolute">
     <parent link="${prefix}_shoulder"/>
     <child link="${prefix}_upper_arm"/>
-    <origin rpy="0 0 0" xyz="0.00 0 0.0"/>
-    <axis xyz="0 ${reflect*1} 0"/>
+    <origin rpy="0 ${reflect*-1.5} 0" xyz="0.00 0 0.0"/>
+    <axis xyz="0 -1 0"/>
     <limit effort="1000.0" lower="-3.14" upper="3.14" velocity="0.5"/>
   </joint>
@@ -49,13 +49,13 @@
     </visual>
 </link>
-  <joint name="${prefix}_elbow" type="revolute">
+  <joint name="${base+5}:${prefix}_elbow" type="revolute">
     <parent link="${prefix}_upper_arm"/>
     <child link="${prefix}_forearm"/>
     <origin rpy="0 0 0" xyz="0.00 0 -0.08"/>
-    <axis xyz="0 ${reflect*1} 0"/>
+    <axis xyz="0 -1 0"/>
     <limit effort="1000.0" lower="-3.14" upper="3.14" velocity="0.5"/>
   </joint>
 </xacro:macro>
-<xacro:macro name="leg" params="prefix reflect">
+<xacro:macro name="leg" params="prefix reflect base">
 <link name="${prefix}_hip">
 	<visual>
@@ -69,9 +69,9 @@
 	</visual>
 </link>
-<joint name="base_to_${prefix}_hip" type="revolute">
+<joint name="${base+7}:base_to_${prefix}_hip" type="revolute">
 	<parent link="base_link"/>
 	<child link="${prefix}_hip"/>
-	<origin rpy="0 0 0" xyz="${reflect*0.030} 0 -0.06"/>
-	<axis xyz="0 0 ${reflect*1}"/>
+	<origin rpy="0 0 ${reflect*-0.70}" xyz="${reflect*0.030} 0 -0.06"/>
+	<axis xyz="0 0 -1"/>
 	<limit effort="1000.0" lower="-3.14" upper="3.14" velocity="0.5"/>
 </joint>
@@ -87,9 +87,9 @@
     </visual>
 </link>
-<joint name="${prefix}_hip_to_split" type="revolute">
+<joint name="${base+9}:${prefix}_hip_to_split" type="revolute">
 <parent link="${prefix}_hip"/>
 <child link="${prefix}_hip_split"/>
 <origin rpy="0 0 0" xyz="0.00 0 0.0"/>
-<axis xyz="0 ${reflect} 0"/>
+<axis xyz="0 1 0"/>
 <limit effort="1000.0" lower="-3.14" upper="3.14" velocity="0.5"/>
 </joint>
@@ -103,9 +103,9 @@
     </visual>
 </link>
-  <joint name="${prefix}_hip_split_to_upper" type="revolute">
+  <joint name="${base+11}:${prefix}_hip_split_to_upper" type="revolute">
     <parent link="${prefix}_hip_split"/>
     <child link="${prefix}_upper_leg"/>
     <origin rpy="0 0 0" xyz="0.00 0 0.0"/>
-    <axis xyz="-1 0 0"/>
+    <axis xyz="${reflect*-1} 0 0"/>
     <limit effort="1000.0" lower="-3.14" upper="3.14" velocity="0.5"/>
   </joint>
@@ -120,9 +120,9 @@
     </visual>
 </link>
-  <joint name="${prefix}_knee" type="revolute">
+  <joint name="${base+13}:${prefix}_knee" type="revolute">
     <parent link="${prefix}_upper_leg"/>
     <child link="${prefix}_calf"/>
     <origin rpy="0 0 0" xyz="0.00 0 -0.08"/>
-    <axis xyz="-1 0 0"/>
+    <axis xyz="${reflect*1} 0 0"/>
     <limit effort="1000.0" lower="-3.14" upper="3.14" velocity="0.5"/>
   </joint>
@@ -136,9 +136,9 @@
     </visual>
 </link>
-  <joint name="${prefix}_ankle" type="revolute">
+  <joint name="${base+15}:${prefix}_ankle" type="revolute">
     <parent link="${prefix}_calf"/>
     <child link="${prefix}_foot"/>
     <origin rpy="0 0 0" xyz="0.00 0 -0.045"/>
-    <axis xyz="-1 0 0"/>
+    <axis xyz="${reflect} 0 0"/>
     <limit effort="1000.0" lower="-3.14" upper="3.14" velocity="0.5"/>
   </joint>
@@ -152,9 +152,9 @@
     </visual>
 </link>
-  <joint name="${prefix}_ankle_roll" type="revolute">
+  <joint name="${base+17}:${prefix}_ankle_roll" type="revolute">
     <parent link="${prefix}_foot"/>
     <child link="${prefix}_foot_pad"/>
     <origin rpy="0 0 0" xyz="0.00 0 -0.03"/>
-    <axis xyz="0 1 0"/>
+    <axis xyz="0 -1 0"/>
     <limit effort="1000.0" lower="-3.14" upper="3.14" velocity="0.5"/>
   </joint>
@@ -167,7 +167,7 @@
 </visual>
 </link>
-<xacro:arm prefix="right" reflect="1"/>
-<xacro:arm prefix="left" reflect="-1"/>
-<xacro:leg prefix="right" reflect="1"/>
-<xacro:leg prefix="left" reflect="-1"/>
+<xacro:arm prefix="right" reflect="1" base="0"/>
+<xacro:arm prefix="left" reflect="-1" base="1"/>
+<xacro:leg prefix="right" reflect="1" base="0"/>
+<xacro:leg prefix="left" reflect="-1" base="1"/>
 </robot>

Commit message: WIP using OpenRAVE's IK solver, doesn't work yet

File: trunk/utilities/ROS/awesomeo_controller/TypeA.xacro (robot description, xacro)
@@ -13,5 +13,5 @@
 </visual>
 </link>
-<joint name="${base+1}:base_to_${prefix}_shoulder" type="revolute">
+<joint name="base_to_${prefix}_shoulder" type="revolute">
 <parent link="base_link"/>
 <child link="${prefix}_shoulder"/>
@@ -32,5 +32,5 @@
     </visual>
 </link>
-  <joint name="${base+3}:${prefix}_shoulder_to_upper" type="revolute">
+  <joint name="${prefix}_shoulder_to_upper" type="revolute">
     <parent link="${prefix}_shoulder"/>
     <child link="${prefix}_upper_arm"/>
@@ -49,5 +49,5 @@
     </visual>
 </link>
-  <joint name="${base+5}:${prefix}_elbow" type="revolute">
+  <joint name="${prefix}_elbow" type="revolute">
     <parent link="${prefix}_upper_arm"/>
     <child link="${prefix}_forearm"/>
@@ -69,5 +69,5 @@
 	</visual>
 </link>
-<joint name="${base+7}:base_to_${prefix}_hip" type="revolute">
+<joint name="base_to_${prefix}_hip" type="revolute">
 	<parent link="base_link"/>
 	<child link="${prefix}_hip"/>
@@ -87,5 +87,5 @@
     </visual>
 </link>
-<joint name="${base+9}:${prefix}_hip_to_split" type="revolute">
+<joint name="${prefix}_hip_to_split" type="revolute">
 <parent link="${prefix}_hip"/>
 <child link="${prefix}_hip_split"/>
@@ -103,5 +103,5 @@
     </visual>
 </link>
-  <joint name="${base+11}:${prefix}_hip_split_to_upper" type="revolute">
+  <joint name="${prefix}_hip_split_to_upper" type="revolute">
     <parent link="${prefix}_hip_split"/>
     <child link="${prefix}_upper_leg"/>
@@ -120,5 +120,5 @@
     </visual>
 </link>
-  <joint name="${base+13}:${prefix}_knee" type="revolute">
+  <joint name="${prefix}_knee" type="revolute">
     <parent link="${prefix}_upper_leg"/>
     <child link="${prefix}_calf"/>
@@ -136,5 +136,5 @@
     </visual>
 </link>
-  <joint name="${base+15}:${prefix}_ankle" type="revolute">
+  <joint name="${prefix}_ankle" type="revolute">
     <parent link="${prefix}_calf"/>
     <child link="${prefix}_foot"/>
@@ -152,5 +152,5 @@
     </visual>
 </link>
-  <joint name="${base+17}:${prefix}_ankle_roll" type="revolute">
+  <joint name="${prefix}_ankle_roll" type="revolute">
     <parent link="${prefix}_foot"/>
     <child link="${prefix}_foot_pad"/>
